File: WavetableController.kicad_sch (KiCad schematic)
At the start: 78 parts, among them J1 Barrel_Jack, J2 SSD1306 OLED, J3 MIDI OUTPUT, J4 AUDIO INPUT, J5 AUDIO OUTPUT, J6 MIDI INPUT, J7 PHONES, P1 Micro_SD_Card_Det2, P2 USB_C31-S-RA-CS2-SMT-BK-T/R, SW1 Power ON/OFF, U1 H11L1, U2 USBLC6-2P6, U3 TPA6110A2DGN, U4 MAX9814

Commit message: Add Round 2 (2026-10) design files, Gerbers and BOM; archive Round 1 files
New set received from Trey on 2026-10-07: .kicad_pcb/.kicad_sch/.kicad_pro
(root), Manifold_Gerbs_2026-10/ (plotted 2026-10-07 12:54 CDT, KiCad 9.0.4)
and the 2026-10-06 BOM. The Round 1 KiCad files and BOM move to
archive/rev1_2026-08/ unchanged. Manifold_Gerb_LedFix/ stays as fab truth
for the boards that physically exist.

Co-Authored-By: Claude Fable 5.1 <noreply@anthropic.com>
Claude-Session: https://claude.ai/code/session_01PLDgQcwfQSF8W6iEm2JuZr
Parts:
- removed C14: 470UF, Capacitor_THT:CP_Radial_D10.0mm_P7.50mm, symbol Device:C_US
- removed C17: 100NF, Capacitor_SMD:C_0603_1608Metric, symbol Device:C
- removed J2: SSD1306 OLED, Retroactive_Custom_Parts:Retroactive_2.42_OLED_I2C, symbol Connector:Conn_01x04_Socket
- added C14: 100NF, Capacitor_SMD:C_0603_1608Metric, symbol Device:C
- added C17, C18, C19, C20, C21, C22: 100UF, Capacitor_SMD:CP_Elec_6.3x7.7, symbol Device:C_US
- added C23: 100NF, Capacitor_THT:C_Axial_L3.8mm_D2.6mm_P7.50mm_Horizontal, symbol Device:C
- added C24: 100UF, Capacitor_THT:CP_Radial_D6.3mm_P2.50mm, symbol Device:C_US
- added C25: 10UF, Capacitor_SMD:C_0603_1608Metric, symbol Device:C
- added C26: 22UF, Capacitor_SMD:C_0603_1608Metric, symbol Device:C
- added D6: D_Schottky, Diode_SMD:D_SOD-323, symbol Device:D_Schottky
- added FB5, FB6, FB7: FerriteBead, Diode_SMD:D_0603_1608Metric, symbol Device:FerriteBead
- added Headphones1: B10k Dual, Retroactive_Custom_Parts:DualGang_Headphone_PTD902-2015K-B103, symbol Device:R_Potentiometer_Dual
- added J8: NHD-2.7-12864WDW3, Retroactive_Custom_Parts:Newhaven2.7_OLED, symbol Connector:Conn_01x20_Pin
- added L1: 2.2UH DFE201610P-2R2M=P2, Inductor_SMD:L_0805_2012Metric, symbol Device:L_Iron
- added R29, R30, R31, R32: 3.3R, Resistor_SMD:R_0603_1608Metric, symbol Device:R
- added R33: 47K, Resistor_SMD:R_0603_1608Metric, symbol Device:R
- added R34: 15K, Resistor_SMD:R_0603_1608Metric, symbol Device:R
- added U6: TPS62172DSG, Package_SON:WSON-8-1EP_2x2mm_P0.5mm_EP0.9x1.6mm_ThermalVias, symbol Regulator_Switching:TPS62172DSG
- C15: value 10UF -> 100UF
Connections:
- net I2C_SCL is gone; now on net ENCR_A: A1.12 (I2C1_SCL)
- net I2C_SDA is gone; now on net ENCR_B: A1.13 (I2C1_SDA)
- net +3V3_A: now also FB2.1, U4.10 (GAIN)
- net +3V3_D: no longer FB2.1, FB4.2, U4.10 (GAIN)
- net AUDIO_OUT_L: now also Headphones1.1; no longer C2.1
- net AUDIO_OUT_R: now also Headphones1.4; no longer C3.1
- net ENCL_CLICK: now also A1.22 (ADC_0); no longer A1.11 (SPI1_PICO)
- net ENCR_A: no longer A1.8 (SPI1_CS)
- net ENCR_B: no longer A1.9 (SPI1_SCK)
- net GND: now also J4.R, C14.2, C17.2, C18.2, C19.2, C20.2, C21.2, C22.2, C23.1, C24.2, C25.2, C26.2, Headphones1.3, Headphones1.6, J8.1 (Pin_1), J8.10 (Pin_10), J8.11 (Pin_11), J8.12 (Pin_12), J8.13 (Pin_13), J8.14 (Pin_14), J8.19 (Pin_19), J8.20 (Pin_20), J8.5 (Pin_5), J8.6 (Pin_6), R34.1, U6.1 (PGND), U6.4 (AGND), U6.9 (PAD)
- net at D2.1 (K), D3.1 (K), FB3.1: now also C14.1; no longer C16.1
- net RES_SPI: now reaches A1.1 (USB_ID)
- net RES_SPI: now also J8.16 (Pin_16)
- net DC_SPI: now reaches A1.28 (ADC_6)
- net DC_SPI: now also J8.4 (Pin_4)
- net +9V_FILT renamed +9V_FLAG
- net +9V_FLAG: now also C21.1, C22.1, FB7.1, R32.2; no longer A1.39 (VIN), C15.1, FB3.2
- net OLED_HOT: no longer names the net of FB4.1
- net OLED_HOT: now also FB3.2
- new net: R33.1, R34.2, U6.5 (FB)
- new net: C15.1, C16.1, D6.2 (A), FB5.2
- new net: C2.1, Headphones1.2
- new net: C3.1, Headphones1.5
- new net: D6.1 (K), FB6.1
- new net: C19.1, FB6.2, R29.1, R31.1
- new net: C20.1, R31.2, R32.1
- new net: C25.1, FB7.2, U6.2 (VIN), U6.3 (EN)
- new net: L1.1, U6.7 (SW)
- new net: C17.1, R29.2, R30.1
- new net: FB4.2, FB5.1
- new net +3V3_OLED: C23.2, C24.1, C26.1, J8.2 (Pin_2), L1.2, R33.2, U6.6 (VOS)
- new net CS_SPI: A1.8 (SPI1_CS), J8.17 (Pin_17)
- new net DSY_VIN: A1.39 (VIN), C18.1, R30.2
- new net SCLK_SPI: A1.9 (SPI1_SCK), J8.7 (Pin_7)
- new net SD_IN_SPI: A1.11 (SPI1_PICO), J8.8 (Pin_8)
Other:
- note added: "Ceramic"
- note added: "NHD-2.7-12864WDW3"
- note added: "OLED 3V3 FILTER"
- note added: "SSD1322"
- note added: "Tantalum"
- note removed: "OLED RC FILT"
- note removed: "Wave Controller Bottom DIY Board"
- moved on the sheet: A1, C1, C10, C11, C12, C13, C2, C3, C4, C5, C6, C7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
